File: mezza.sch (KiCad schematic (older format))
At the start: 15 parts, among them CON1 USB-MINI-B, P1 CONN_02X20, P2 CONN_02X20, U1 TXS0108E, U2 FT230XS, U3 CJT1117-3.3

Commit message: Flip USB Connector, Rename GPIO Signals, Remove Level Shifter
The USB connector has been flipped so that the data signals are cleaner.
Regulator has been changed from CJT1117-3.3 (which regulates to 3.3V)
to XC6206 (which regulates to 1.8V).
GPIO-A & GPIO-B have been changed to "GPIO_A" & "GPIO_B" to keep consistent
with rest of signal names.
Level shifter has been removed temporarily.

Signed-Off-By: Sophie Haynes<sophie.haynes@linaro.org>
Parts:
- removed U1: TXS0108E, Housings_SSOP:TSSOP-20_4.4x6.5mm_Pitch0.65mm, symbol TXS0108E
- U3: value CJT1117-3.3 -> XC6206
Connections:
- net labels added: GPIO_A, GPIO_B
- net labels removed: +3.3V, GPIO-A, GPIO-B
- wire segments 146 -> 133
- no-connect marks 55 -> 45
Other:
- note removed: "LEVEL\nSHIFTER"
- moved on the sheet: C3, CON1, R1, R2, U2

Commit message: Add LED Indication for RX/TX
An LED wired to CBUS0 & CBUS1 has been added to show RX/TX activity.
Connected to +5V and both lines have 220R.

Signed-Off-By: Sophie Haynes<sophie.haynes@linaro.org>
Parts:
- added D?: RX, symbol Led_Small
- added D?: TX, symbol Led_Small
- added R? (x2): 220R, symbol R
Connections:
- net labels added: CBUS0, CBUS1
- wire segments 133 -> 142
- no-connect marks 45 -> 43
Changed lines of the file:
@@
 	1    0    0    -1
 $EndComp
-NoConn ~ 5200 5500
-NoConn ~ 5200 5600
 Wire Wire Line
 	1850 5450 2400 5450
@@
 NoConn ~ 5200 4900
 NoConn ~ 5200 5000
+Text GLabel 5350 5600 2    60   Input ~ 0
+CBUS1
+Text GLabel 5350 5500 2    60   Input ~ 0
+CBUS0
+Wire Wire Line
+	5350 5500 5200 5500
+Wire Wire Line
+	5350 5600 5200 5600
+Text GLabel 750  7300 3    60   Input ~ 0
+CBUS1
+Text GLabel 1100 7300 3    60   Input ~ 0
+CBUS0
+$Comp
+L Led_Small D?
+U 1 1 5659A589
+P 750 6950
+F 0 "D?" H 700 7075 50  0000 L CNN
+F 1 "RX" H 575 6850 50  0000 L CNN
+F 2 "" V 750 6950 60  0000 C CNN
+F 3 "" V 750 6950 60  0000 C CNN
+	1    750  6950
+	0    -1   -1   0
+$EndComp
+$Comp
+L Led_Small D?
+U 1 1 5659A5E7
+P 1100 6950
+F 0 "D?" H 1050 7075 50  0000 L CNN
+F 1 "TX" H 925 6850 50  0000 L CNN
+F 2 "" V 1100 6950 60  0000 C CNN
+F 3 "" V 1100 6950 60  0000 C CNN
+	1    1100 6950
+	0    -1   -1   0
+$EndComp
+Wire Wire Line
+	750  7050 750  7300
+Wire Wire Line
+	1100 7050 1100 7300
+$Comp
+L R R?
+U 1 1 5659A75D
+P 750 6450
+F 0 "R?" V 830 6450 50  0000 C CNN
+F 1 "220R" V 750 6450 50  0000 C CNN
+F 2 "" V 680 6450 30  0000 C CNN
+F 3 "" H 750 6450 30  0000 C CNN
+	1    750  6450
+	1    0    0    -1
+$EndComp
+$Comp
+L R R?
+U 1 1 5659A7A3
+P 1100 6450
+F 0 "R?" V 1180 6450 50  0000 C CNN
+F 1 "220R" V 1100 6450 50  0000 C CNN
+F 2 "" V 1030 6450 30  0000 C CNN
+F 3 "" H 1100 6450 30  0000 C CNN
+	1    1100 6450
+	1    0    0    -1
+$EndComp
+$Comp
+L +5V #PWR?
+U 1 1 5659A808
+P 950 6150
+F 0 "#PWR?" H 950 6000 50  0001 C CNN
+F 1 "+5V" H 950 6290 50  0000 C CNN
+F 2 "" H 950 6150 60  0000 C CNN
+F 3 "" H 950 6150 60  0000 C CNN
+	1    950  6150
+	1    0    0    -1
+$EndComp
+Wire Wire Line
+	750  6600 750  6850
+Wire Wire Line
+	1100 6600 1100 6850
+Wire Wire Line
+	750  6150 1100 6150
+Wire Wire Line
+	1100 6150 1100 6300
+Wire Wire Line
+	750  6300 750  6150
+Connection ~ 950  6150
 $EndSCHEMATC

Commit message: Insert Resistors Between PWR/RST
220R resistors have been between PWR_BTN and RST_BTN to provide
protection. Schematic has been annotated accordingly.

Signed-Off-By: Sophie Haynes<sophie.haynes@linaro.org>
Parts:
- added R5, R6: 220R, symbol R
- gave numbers to parts that had none: 4
Connections:
- wire segments 142 -> 146
Changed lines of the file:
@@
 $EndComp
 $Comp
-L GND #PWR02
+L GND #PWR6
 U 1 1 55BEB06A
 P 1200 3950
-F 0 "#PWR02" H 1200 3700 50  0001 C CNN
+F 0 "#PWR6" H 1200 3700 50  0001 C CNN
 F 1 "GND" H 1200 3800 50  0000 C CNN
 F 2 "" H 1200 3950 60  0000 C CNN
@@
 $EndComp
 $Comp
-L GND #PWR03
+L GND #PWR7
 U 1 1 55BEAA68
 P 1500 750
-F 0 "#PWR03" H 1500 500 50  0001 C CNN
+F 0 "#PWR7" H 1500 500 50  0001 C CNN
 F 1 "GND" H 1500 600 50  0000 C CNN
 F 2 "" H 1500 750 60  0000 C CNN
@@
 $EndComp
 $Comp
-L GND #PWR04
+L GND #PWR8
 U 1 1 55BEA10A
 P 1550 2800
-F 0 "#PWR04" H 1550 2550 50  0001 C CNN
+F 0 "#PWR8" H 1550 2550 50  0001 C CNN
 F 1 "GND" H 1550 2650 50  0000 C CNN
 F 2 "" H 1550 2800 60  0000 C CNN
@@
 $EndComp
 $Comp
-L GND #PWR05
+L GND #PWR12
 U 1 1 55BEA0BC
 P 2250 2800
-F 0 "#PWR05" H 2250 2550 50  0001 C CNN
+F 0 "#PWR12" H 2250 2550 50  0001 C CNN
 F 1 "GND" H 2250 2650 50  0000 C CNN
 F 2 "" H 2250 2800 60  0000 C CNN
@@
 SYS_DCIN
 $Comp
-L GND #PWR06
+L GND #PWR13
 U 1 1 55D43BD4
 P 2300 750
-F 0 "#PWR06" H 2300 500 50  0001 C CNN
+F 0 "#PWR13" H 2300 500 50  0001 C CNN
 F 1 "GND" H 2300 600 50  0000 C CNN
 F 2 "" H 2300 750 60  0000 C CNN
@@
 $EndComp
 $Comp
-L +1V8 #PWR07
+L +1V8 #PWR5
 U 1 1 55D43CFB
 P 1000 2550
-F 0 "#PWR07" H 1000 2400 50  0001 C CNN
+F 0 "#PWR5" H 1000 2400 50  0001 C CNN
 F 1 "+1V8" H 1000 2690 50  0000 C CNN
 F 2 "" H 1000 2550 60  0000 C CNN
@@
 $EndComp
 $Comp
-L +5V #PWR08
+L +5V #PWR3
 U 1 1 55D440FD
 P 800 2550
-F 0 "#PWR08" H 800 2400 50  0001 C CNN
+F 0 "#PWR3" H 800 2400 50  0001 C CNN
 F 1 "+5V" H 800 2690 50  0000 C CNN
 F 2 "" H 800 2550 60  0000 C CNN
@@
 I2C0_SCL
 $Comp
-L GND #PWR09
+L GND #PWR22
 U 1 1 55D481C7
 P 3700 750
-F 0 "#PWR09" H 3700 500 50  0001 C CNN
+F 0 "#PWR22" H 3700 500 50  0001 C CNN
 F 1 "GND" H 3700 600 50  0000 C CNN
 F 2 "" H 3700 750 60  0000 C CNN
@@
 UART_TX
 $Comp
-L GND #PWR010
+L GND #PWR23
 U 1 1 55D481CF
 P 3750 2800
-F 0 "#PWR010" H 3750 2550 50  0001 C CNN
+F 0 "#PWR23" H 3750 2550 50  0001 C CNN
 F 1 "GND" H 3750 2650 50  0000 C CNN
 F 2 "" H 3750 2800 60  0000 C CNN
@@
 $EndComp
 $Comp
-L GND #PWR011
+L GND #PWR25
 U 1 1 55D481D5
 P 4450 2800
-F 0 "#PWR011" H 4450 2550 50  0001 C CNN
+F 0 "#PWR25" H 4450 2550 50  0001 C CNN
 F 1 "GND" H 4450 2650 50  0000 C CNN
 F 2 "" H 4450 2800 60  0000 C CNN
@@
 SYS_DCIN
 $Comp
-L GND #PWR012
+L GND #PWR26
 U 1 1 55D48218
 P 4500 750
-F 0 "#PWR012" H 4500 500 50  0001 C CNN
+F 0 "#PWR26" H 4500 500 50  0001 C CNN
 F 1 "GND" H 4500 600 50  0000 C CNN
 F 2 "" H 4500 750 60  0000 C CNN
@@
 $EndComp
 $Comp
-L +1V8 #PWR013
+L +1V8 #PWR21
 U 1 1 55D4822C
 P 3200 2550
-F 0 "#PWR013" H 3200 2400 50  0001 C CNN
+F 0 "#PWR21" H 3200 2400 50  0001 C CNN
 F 1 "+1V8" H 3200 2690 50  0000 C CNN
 F 2 "" H 3200 2550 60  0000 C CNN
@@
 $EndComp
 $Comp
-L +5V #PWR014
+L +5V #PWR17
 U 1 1 55D48233
 P 3000 2550
-F 0 "#PWR014" H 3000 2400 50  0001 C CNN
+F 0 "#PWR17" H 3000 2400 50  0001 C CNN
 F 1 "+5V" H 3000 2690 50  0000 C CNN
 F 2 "" H 3000 2550 60  0000 C CNN
@@
 $EndComp
 $Comp
-L +1V8 #PWR015
+L +1V8 #PWR9
 U 1 1 55D44684
 P 1600 3300
-F 0 "#PWR015" H 1600 3150 50  0001 C CNN
+F 0 "#PWR9" H 1600 3150 50  0001 C CNN
 F 1 "+1V8" H 1600 3440 50  0000 C CNN
 F 2 "" H 1600 3300 60  0000 C CNN
@@
 Text Notes 1000 4250 0    60   ~ 0
 Regulator
-Text GLabel 5350 5700 2    60   Input ~ 0
+Text GLabel 6200 5700 2    60   Input ~ 0
 PWR_BTN_N
 Text GLabel 4450 1100 2    60   Input ~ 0
@@
 GPIO_B
 $Comp
-L GND #PWR017
+L GND #PWR24
 U 1 1 563E2DA1
 P 4300 6650
-F 0 "#PWR017" H 4300 6400 50  0001 C CNN
+F 0 "#PWR24" H 4300 6400 50  0001 C CNN
 F 1 "GND" H 4300 6500 50  0000 C CNN
 F 2 "" H 4300 6650 60  0000 C CNN
@@
 NoConn ~ 4450 2500
 $Comp
-L +1V8 #PWR018
+L +1V8 #PWR18
 U 1 1 56432A36
 P 3150 4650
-F 0 "#PWR018" H 3150 4500 50  0001 C CNN
+F 0 "#PWR18" H 3150 4500 50  0001 C CNN
 F 1 "+1V8" H 3150 4790 50  0000 C CNN
 F 2 "" H 3150 4650 60  0000 C CNN
@@
 Text GLabel 3700 1200 0    60   Input ~ 0
 UART_RX
-Text GLabel 5350 5800 2    60   Input ~ 0
+Text GLabel 6200 5900 2    60   Input ~ 0
 RST_BTN_N
 $Comp
-L +3V3_FTDI #PWR019
+L +3V3_FTDI #PWR19
 U 1 1 564330C0
 P 3150 5300
-F 0 "#PWR019" H 3150 5150 50  0001 C CNN
+F 0 "#PWR19" H 3150 5150 50  0001 C CNN
 F 1 "+3V3_FTDI" H 3150 5440 50  0000 C CNN
 F 2 "" H 3150 5300 60  0000 C CNN
@@
 NoConn ~ 1850 5300
 $Comp
-L GND #PWR020
+L GND #PWR11
 U 1 1 564CDC20
 P 2000 5600
-F 0 "#PWR020" H 2000 5350 50  0001 C CNN
+F 0 "#PWR11" H 2000 5350 50  0001 C CNN
 F 1 "GND" H 2000 5450 50  0000 C CNN
 F 2 "" H 2000 5600 60  0000 C CNN
@@
 $EndComp
 $Comp
-L GND #PWR021
+L GND #PWR2
 U 1 1 564CDC85
 P 750 5550
-F 0 "#PWR021" H 750 5300 50  0001 C CNN
+F 0 "#PWR2" H 750 5300 50  0001 C CNN
 F 1 "GND" H 750 5400 50  0000 C CNN
 F 2 "" H 750 5550 60  0000 C CNN
@@
 $EndComp
 $Comp
-L VBUS #PWR022
+L VBUS #PWR10
 U 1 1 564CEA94
 P 1900 4750
-F 0 "#PWR022" H 1900 4850 30  0001 C CNN
+F 0 "#PWR10" H 1900 4850 30  0001 C CNN
 F 1 "VBUS" H 1900 4860 30  0000 C CNN
 F 2 "" H 1900 4750 60  0000 C CNN
@@
 $EndComp
 $Comp
-L VBUS #PWR023
+L VBUS #PWR16
 U 1 1 564CEB6E
 P 2950 4750
-F 0 "#PWR023" H 2950 4850 30  0001 C CNN
+F 0 "#PWR16" H 2950 4850 30  0001 C CNN
 F 1 "VBUS" H 2950 4860 30  0000 C CNN
 F 2 "" H 2950 4750 60  0000 C CNN
@@
 $EndComp
 $Comp
-L VBUS #PWR024
+L VBUS #PWR14
 U 1 1 564CECA3
 P 2400 3300
-F 0 "#PWR024" H 2400 3400 30  0001 C CNN
+F 0 "#PWR14" H 2400 3400 30  0001 C CNN
 F 1 "VBUS" H 2400 3410 30  0000 C CNN
 F 2 "" H 2400 3300 60  0000 C CNN
@@
 $EndComp
 $Comp
-L GND #PWR025
+L GND #PWR15
 U 1 1 564CEDC1
 P 2400 3950
-F 0 "#PWR025" H 2400 3700 50  0001 C CNN
+F 0 "#PWR15" H 2400 3700 50  0001 C CNN
 F 1 "GND" H 2400 3800 50  0000 C CNN
 F 2 "" H 2400 3950 60  0000 C CNN
@@
 PWR_BTN_N
 $Comp
-L GND #PWR027
+L GND #PWR20
 U 1 1 56530F98
 P 3150 6600
-F 0 "#PWR027" H 3150 6350 50  0001 C CNN
+F 0 "#PWR20" H 3150 6350 50  0001 C CNN
 F 1 "GND" H 3150 6450 50  0000 C CNN
 F 2 "" H 3150 6600 60  0000 C CNN
@@
 	3150 5300 3150 6050
 Wire Wire Line
-	5350 5700 5200 5700
-Wire Wire Line
-	5350 5800 5200 5800
+	5200 5700 5750 5700
+Wire Wire Line
+	5200 5800 5500 5800
 Wire Wire Line
 	3350 4650 3150 4650
@@
 Connection ~ 2400 5000
 $Comp
-L +3V3 #PWR016
+L +3V3 #PWR1
 U 1 1 55D4457B
 P 750 3300
-F 0 "#PWR016" H 750 3150 50  0001 C CNN
+F 0 "#PWR1" H 750 3150 50  0001 C CNN
 F 1 "+3V3" H 750 3440 50  0000 C CNN
 F 2 "" H 750 3300 60  0000 C CNN
@@
 CBUS0
 $Comp
-L Led_Small D?
+L Led_Small D1
 U 1 1 5659A589
 P 750 6950
-F 0 "D?" H 700 7075 50  0000 L CNN
+F 0 "D1" H 700 7075 50  0000 L CNN
 F 1 "RX" H 575 6850 50  0000 L CNN
 F 2 "" V 750 6950 60  0000 C CNN
@@
 $EndComp
 $Comp
-L Led_Small D?
+L Led_Small D2
 U 1 1 5659A5E7
 P 1100 6950
-F 0 "D?" H 1050 7075 50  0000 L CNN
+F 0 "D2" H 1050 7075 50  0000 L CNN
 F 1 "TX" H 925 6850 50  0000 L CNN
 F 2 "" V 1100 6950 60  0000 C CNN
@@
 	1100 7050 1100 7300
 $Comp
-L R R?
+L R R3
 U 1 1 5659A75D
 P 750 6450
-F 0 "R?" V 830 6450 50  0000 C CNN
+F 0 "R3" V 830 6450 50  0000 C CNN
 F 1 "220R" V 750 6450 50  0000 C CNN
 F 2 "" V 680 6450 30  0000 C CNN
@@
 $EndComp
 $Comp
-L R R?
+L R R4
 U 1 1 5659A7A3
 P 1100 6450
-F 0 "R?" V 1180 6450 50  0000 C CNN
+F 0 "R4" V 1180 6450 50  0000 C CNN
 F 1 "220R" V 1100 6450 50  0000 C CNN
 F 2 "" V 1030 6450 30  0000 C CNN
@@
 $EndComp
 $Comp
-L +5V #PWR?
+L +5V #PWR4
 U 1 1 5659A808
 P 950 6150
-F 0 "#PWR?" H 950 6000 50  0001 C CNN
+F 0 "#PWR4" H 950 6000 50  0001 C CNN
 F 1 "+5V" H 950 6290 50  0000 C CNN
 F 2 "" H 950 6150 60  0000 C CNN
@@
 	750  6300 750  6150
 Connection ~ 950  6150
+$Comp
+L R R6
+U 1 1 5659B859
+P 5900 5900
+F 0 "R6" V 5980 5900 50  0000 C CNN
+F 1 "220R" V 5900 5900 50  0000 C CNN
+F 2 "" V 5830 5900 30  0000 C CNN
+F 3 "" H 5900 5900 30  0000 C CNN
+	1    5900 5900
+	0    1    1    0
+$EndComp
+$Comp
+L R R5
+U 1 1 5659B8C3
+P 5900 5700
+F 0 "R5" V 5980 5700 50  0000 C CNN
+F 1 "220R" V 5900 5700 50  0000 C CNN
+F 2 "" V 5830 5700 30  0000 C CNN
+F 3 "" H 5900 5700 30  0000 C CNN
+	1    5900 5700
+	0    1    1    0
+$EndComp
+Wire Wire Line
+	6050 5700 6200 5700
+Wire Wire Line
+	6200 5900 6050 5900
+Wire Wire Line
+	5750 5900 5500 5900
+Wire Wire Line
+	5500 5900 5500 5800
 $EndSCHEMATC

Commit message: Add PWR LED, Remove 2nd Expansion Conn. Footprint
LED's for each power rail have been added (+5V, +3V3, +1V8) to show when
each is live.
The footprint for the second expansion connector has been removed so that it
is now a standard through-hole port.

Signed-Off-By: Sophie Haynes <sophie.haynes@linaro.org>
Parts:
- added D3, D4, D5: Led_Small, symbol Led_Small
- added R7, R8, R9: 220R, symbol R
- P2: footprint mezza:Pin_Header_SMD_2x20_Pitch2mm -> (none)
Connections:
- wire segments 146 -> 155
Other:
- note added: "PWR LED Indicators"
- note added: "RX/TX LED Indicators"
- moved on the sheet: C3, CON1, D1, D2, R1, R2, R3, R4, R5, U2

Commit message: Label All Signals on Expansion Conn, Connect FTDI to UART1
All the signals have been labeled to make it easier when starting a new
project with this schematic.
UART0 was previously named "UART"; this has been changed to "UART0" to prevent
confusion as UART1 has been added.
FTDI is now connected to UART1 rather than UART0

Signed-off-by: Sophie Haynes<sophie.haynes@linaro.org>
Connections:
- net labels added: GPIO_C, GPIO_D, GPIO_E, GPIO_F, GPIO_G, GPIO_H, GPIO_I, GPIO_J, GPIO_K, GPIO_L, PCM_CLK, PCM_DI, PCM_DO, PCM_FS, SPIO_CS, SPIO_DIN, SPIO_DOUT, SPIO_SCL, UART0_CTS, UART0_RTS, UART0_RX, UART0_TX, UART1_RX, UART1_TX
- no-connect marks 43 -> 3
Other:
- moved on the sheet: R6

Commit message: Add 3v3_F Component & Change Power Signals According
A new power component has been added to the mezza library (3v3_F). This is to
replace '3v3_FTDI' and serve as an individual power source for specific
components.

Signed-off-by: Sophie Haynes<sophie.haynes@linaro.org>
Connections:
- net labels added: +3V3_F
- net labels removed: +3V3, +3V3_FTDI
Changed lines of the file:
@@
 RST_BTN_N
 $Comp
-L +3V3_FTDI #PWR017
+L +3V3_F #PWR017
 U 1 1 564330C0
 P 3150 5100
 F 0 "#PWR017" H 3150 4950 50  0001 C CNN
-F 1 "+3V3_FTDI" H 3150 5240 50  0000 C CNN
+F 1 "+3V3_F" H 3150 5240 50  0000 C CNN
 F 2 "" H 3150 5100 60  0000 C CNN
 F 3 "" H 3150 5100 60  0000 C CNN
@@
 	2300 6400 2300 6650
 $Comp
-L +3V3 #PWR031
+L +3V3_F #PWR031
 U 1 1 5659D6C2
 P 2300 5950
 F 0 "#PWR031" H 2300 5800 50  0001 C CNN
-F 1 "+3V3" H 2300 6090 50  0000 C CNN
+F 1 "+3V3_F" H 2300 6090 50  0000 C CNN
 F 2 "" H 2300 5950 60  0000 C CNN
 F 3 "" H 2300 5950 60  0000 C CNN
@@
 Text GLabel 4450 2500 2    60   Input ~ 0
 GPIO_L
+$Comp
+L +3V3_F #PWR?
+U 1 1 56685B3D
+P 750 3300
+F 0 "#PWR?" H 750 3150 50  0001 C CNN
+F 1 "+3V3_F" H 750 3440 50  0000 C CNN
+F 2 "" H 750 3300 60  0000 C CNN
+F 3 "" H 750 3300 60  0000 C CNN
+	1    750  3300
+	1    0    0    -1
+$EndComp
 $EndSCHEMATC
