File: boards/kicad/proto-mezzanine/proto-mezzanine.sch (KiCad schematic (older format))
At the start: 5 parts, among them J1 CONN_01X04, J2 CONN_01X04, J3 CONN_01X02, J4 CONN_01X12, P1 CONN_02X20

Commit message: Proto mezzanine updated to v1.4
Changes
- Labled i2c -> i2c0
- Removed pads from lower third to stop interference with ports on base board
- Reduced size of the board on the Y-axis

Signed-off-by: Sahaj Sarup <sahajsarup@linaro.org>
Parts:
- J1, J2: symbol CONN_01X04 -> proto-mezzanine-rescue:CONN_01X04
- J3: symbol CONN_01X02 -> proto-mezzanine-rescue:CONN_01X02
- J4: symbol CONN_01X12 -> proto-mezzanine-rescue:CONN_01X12
- P1: symbol CONN_02X20 -> 96boards:CONN_02X20
Connections:
- wire segments 69 -> 70
Changed lines of the file:
@@
-EESchema Schematic File Version 2
-LIBS:power
-LIBS:device
-LIBS:transistors
-LIBS:conn
-LIBS:linear
-LIBS:regul
-LIBS:74xx
-LIBS:cmos4000
-LIBS:adc-dac
-LIBS:memory
-LIBS:xilinx
-LIBS:microcontrollers
-LIBS:dsp
-LIBS:microchip
-LIBS:analog_switches
-LIBS:motorola
-LIBS:texas
-LIBS:intel
-LIBS:audio
-LIBS:interface
-LIBS:digital-audio
-LIBS:philips
-LIBS:display
-LIBS:cypress
-LIBS:siliconi
-LIBS:opto
-LIBS:atmel
-LIBS:contrib
-LIBS:valves
-LIBS:96boards
+EESchema Schematic File Version 4
 LIBS:proto-mezzanine-cache
 EELAYER 26 0
@@
 encoding utf-8
 Sheet 1 1
-Title "PROTO MEZZANINE V1.3"
-Date "14 Aug 2015"
+Title "PROTO MEZZANINE V1.4"
+Date "2019-02-21"
 Rev "A"
 Comp "Barry Byford"
 Comment1 "Converted to KiCAD by Michael Welling"
-Comment2 ""
+Comment2 "V1.4 by Sahaj Sarup"
 Comment3 ""
 Comment4 ""
 $EndDescr
 $Comp
-L GND #PWR07
+L power:GND #PWR07
 U 1 1 55BEAA68
 P 4050 2500
@@
 $EndComp
 $Comp
-L GND #PWR08
+L power:GND #PWR08
 U 1 1 55BEA10A
 P 4100 4550
@@
 $EndComp
 $Comp
-L GND #PWR09
+L power:GND #PWR09
 U 1 1 55BEA0BC
 P 4800 4550
@@
 SYS_DCIN
 $Comp
-L GND #PWR010
+L power:GND #PWR010
 U 1 1 55D43BD4
 P 4850 2500
@@
 $EndComp
 $Comp
-L CONN_02X20 P1
+L 96boards:CONN_02X20 P1
 U 1 1 55D44709
 P 4450 3600
@@
 $EndComp
 $Comp
-L +1V8 #PWR011
+L power:+1V8 #PWR011
 U 1 1 55D43CFB
 P 3550 4300
@@
 $EndComp
 $Comp
-L +5V #PWR012
+L power:+5V #PWR012
 U 1 1 55D440FD
 P 3350 4300
@@
 	4700 4350 4750 4350
 Wire Wire Line
-	4700 4450 4800 4450
+	4700 4450 4750 4450
 Wire Wire Line
 	4050 2450 4050 2500
@@
 	4200 3050 4050 3050
 $Comp
-L CONN_01X04 J1
+L proto-mezzanine-rescue:CONN_01X04 J1
 U 1 1 5987B130
 P 7450 2750
@@
 $EndComp
 $Comp
-L CONN_01X04 J2
+L proto-mezzanine-rescue:CONN_01X04 J2
 U 1 1 5987B1FD
 P 7450 3250
@@
 $EndComp
 $Comp
-L CONN_01X02 J3
+L proto-mezzanine-rescue:CONN_01X02 J3
 U 1 1 5987B24F
 P 7450 3650
@@
 GPIO_L
 $Comp
-L CONN_01X12 J4
+L proto-mezzanine-rescue:CONN_01X12 J4
 U 1 1 5987B843
 P 7450 4450
@@
 Wire Notes Line
 	4600 5900 4600 5500
+Wire Wire Line
+	4750 4450 4800 4450
 $EndSCHEMATC
