File: template/eaglecad/mezza.brd (EAGLE design)
At the start: 85 x 54 mm, 3 parts, among them J1 55510-140LF, J2 61083-063402LF

Commit message: update Eagle schematic and library
Parts:
- J1: value 55510-140LF -> 57202-G52-20LF; device mezza:55510-140LF -> mezza:57202-G52-20LF
Changed lines of the file:
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@@
 <?xml version="1.0" encoding="utf-8"?>
 <!DOCTYPE eagle SYSTEM "eagle.dtd">
-<eagle version="6.6.0">
+<eagle version="9.5.2">
 <drawing>
 <settings>
-<setting alwaysvectorfont="no"/>
+<setting alwaysvectorfont="yes"/>
+<setting keepoldvectorfont="yes"/>
 <setting verticaltext="up"/>
 </settings>
@@
 <param name="dpMaxLengthDifference" value="10mm"/>
 <param name="dpGapFactor" value="2.5"/>
-<param name="checkGrid" value="0"/>
 <param name="checkAngle" value="0"/>
 <param name="checkFont" value="1"/>
 <param name="checkRestrict" value="1"/>
+<param name="checkStop" value="0"/>
+<param name="checkValues" value="0"/>
+<param name="checkNames" value="1"/>
+<param name="checkWireStubs" value="1"/>
+<param name="checkPolygonWidth" value="0"/>
 <param name="useDiameter" value="13"/>
 <param name="maxErrors" value="50"/>
@@
 <pass name="Default">
 <param name="RoutingGrid" value="50mil"/>
+<param name="AutoGrid" value="1"/>
+<param name="Efforts" value="0"/>
+<param name="TopRouterVariant" value="1"/>
 <param name="tpViaShape" value="round"/>
 <param name="PrefDir.1" value="|"/>
@@
 </autorouter>
 <elements>
-<element name="PCB1" library="mezza" package="DRAGONBOARD410C" value="DB410C-PCB-FOOTPRINT" x="0" y="0"/>
-<element name="J1" library="mezza" package="55510-140LF" value="55510-140LF" x="29" y="50" smashed="yes" rot="MR180">
+<element name="PCB1" library="mezza" package="DRAGONBOARD410C" value="DB410C-PCB-FOOTPRINT" x="0" y="0" smashed="yes"/>
+<element name="J1" library="mezza" package="57202-G52-20LF" value="57202-G52-20LF" x="29" y="50" smashed="yes" rot="MR180">
 <attribute name="NAME" x="8.68" y="51" size="1.27" layer="26" rot="MR270"/>
 </element>
@@
 <contactref element="J2" pad="P$58"/>
 <wire x1="81" y1="18.5" x2="81" y2="50" width="0" layer="19" extent="1-1"/>
-<wire x1="48" y1="52.5" x2="81" y2="50" width="0" layer="19" extent="16-16"/>
-<wire x1="48" y1="47.5" x2="48" y2="52.5" width="0" layer="19" extent="16-16"/>
-<wire x1="43.55" y1="17.65" x2="48" y2="47.5" width="0" layer="19" extent="16-16"/>
+<wire x1="48" y1="52" x2="81" y2="50" width="0" layer="19" extent="16-16"/>
+<wire x1="48" y1="48" x2="48" y2="52" width="0" layer="19" extent="16-16"/>
+<wire x1="43.55" y1="17.65" x2="48" y2="48" width="0" layer="19" extent="16-16"/>
 <wire x1="41.15" y1="17.65" x2="43.55" y2="17.65" width="0" layer="19" extent="16-16"/>
 <wire x1="38.75" y1="17.65" x2="41.15" y2="17.65" width="0" layer="19" extent="16-16"/>
@@
 <wire x1="25.95" y1="13.25" x2="28.35" y2="13.25" width="0" layer="19" extent="16-16"/>
 <wire x1="4" y1="18.5" x2="22.75" y2="17.65" width="0" layer="19" extent="16-16"/>
-<wire x1="10" y1="47.5" x2="4" y2="18.5" width="0" layer="19" extent="16-16"/>
-<wire x1="10" y1="52.5" x2="10" y2="47.5" width="0" layer="19" extent="16-16"/>
-<wire x1="4" y1="50" x2="10" y2="47.5" width="0" layer="19" extent="16-16"/>
+<wire x1="10" y1="48" x2="4" y2="18.5" width="0" layer="19" extent="16-16"/>
+<wire x1="10" y1="52" x2="10" y2="48" width="0" layer="19" extent="16-16"/>
+<wire x1="4" y1="50" x2="10" y2="48" width="0" layer="19" extent="16-16"/>
 </signal>
 <signal name="UART0_CTS">
@@
 <contactref element="J1" pad="P$36"/>
 <contactref element="J1" pad="P$38"/>
-<wire x1="44" y1="52.5" x2="46" y2="52.5" width="0" layer="19" extent="16-16"/>
+<wire x1="44" y1="52" x2="46" y2="52" width="0" layer="19" extent="16-16"/>
 </signal>
 <signal name="SD_DAT1">
@@
 </signal>
 </signals>
+<mfgpreviewcolors>
+<mfgpreviewcolor name="soldermaskcolor" color="0xC8008000"/>
+<mfgpreviewcolor name="silkscreencolor" color="0xFFFEFEFE"/>
+<mfgpreviewcolor name="backgroundcolor" color="0xFF282828"/>
+<mfgpreviewcolor name="coppercolor" color="0xFFFFBF00"/>
+<mfgpreviewcolor name="substratecolor" color="0xFF786E46"/>
+</mfgpreviewcolors>
 </board>
 </drawing>
