File: template/eaglecad/mezza.sch (EAGLE design)
At the start: 3 parts, among them J1 55510-140LF, J2 61083-063402LF

Commit message: update Eagle schematic and library
Parts:
- J1: value 55510-140LF -> 57202-G52-20LF; device mezza:55510-140LF -> mezza:57202-G52-20LF
Changed lines of the file:
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@@
 <?xml version="1.0" encoding="utf-8"?>
 <!DOCTYPE eagle SYSTEM "eagle.dtd">
-<eagle version="6.6.0">
+<eagle version="9.5.2">
 <drawing>
 <settings>
-<setting alwaysvectorfont="no"/>
+<setting alwaysvectorfont="yes"/>
+<setting keepoldvectorfont="yes"/>
 <setting verticaltext="up"/>
 </settings>
@@
 <parts>
 <part name="PCB1" library="mezza" deviceset="DB410C-PCB-FOOTPRINT" device=""/>
-<part name="J1" library="mezza" deviceset="55510-140LF" device=""/>
+<part name="J1" library="mezza" deviceset="57202-G52-20LF" device=""/>
 <part name="J2" library="mezza" deviceset="61083-063402LF" device=""/>
 <part name="SUPPLY1" library="supply2" deviceset="GND" device=""/>
@@
 <attribute name="VALUE" x="55.88" y="0" size="2.54" layer="96"/>
 </instance>
-<instance part="SUPPLY7" gate="GND" x="48.26" y="-5.08"/>
-<instance part="SUPPLY8" gate="GND" x="88.9" y="-5.08"/>
+<instance part="SUPPLY7" gate="GND" x="48.26" y="-5.08" smashed="yes">
+<attribute name="VALUE" x="46.355" y="-8.255" size="1.778" layer="96"/>
+</instance>
+<instance part="SUPPLY8" gate="GND" x="88.9" y="-5.08" smashed="yes">
+<attribute name="VALUE" x="86.995" y="-8.255" size="1.778" layer="96"/>
+</instance>
 <instance part="J1" gate="G$1" x="-66.04" y="48.26" smashed="yes">
 <attribute name="NAME" x="-68.58" y="78.74" size="2.54" layer="95"/>
 <attribute name="VALUE" x="-76.2" y="17.78" size="2.54" layer="96"/>
 </instance>
-<instance part="SUPPLY2" gate="GND" x="-83.82" y="81.28" rot="R180"/>
-<instance part="SUPPLY3" gate="GND" x="-83.82" y="12.7"/>
-<instance part="SUPPLY5" gate="GND" x="-48.26" y="81.28" rot="R180"/>
-<instance part="SUPPLY6" gate="GND" x="-48.26" y="12.7"/>
-<instance part="PCB1" gate="G$1" x="-63.5" y="-27.94"/>
-<instance part="SUPPLY1" gate="GND" x="-76.2" y="-48.26"/>
-<instance part="FRAME3" gate="G$1" x="-129.54" y="-68.58"/>
+<instance part="SUPPLY2" gate="GND" x="-83.82" y="81.28" smashed="yes" rot="R180">
+<attribute name="VALUE" x="-81.915" y="84.455" size="1.778" layer="96" rot="R180"/>
+</instance>
+<instance part="SUPPLY3" gate="GND" x="-83.82" y="12.7" smashed="yes">
+<attribute name="VALUE" x="-85.725" y="9.525" size="1.778" layer="96"/>
+</instance>
+<instance part="SUPPLY5" gate="GND" x="-48.26" y="81.28" smashed="yes" rot="R180">
+<attribute name="VALUE" x="-46.355" y="84.455" size="1.778" layer="96" rot="R180"/>
+</instance>
+<instance part="SUPPLY6" gate="GND" x="-48.26" y="12.7" smashed="yes">
+<attribute name="VALUE" x="-50.165" y="9.525" size="1.778" layer="96"/>
+</instance>
+<instance part="PCB1" gate="G$1" x="-63.5" y="-27.94" smashed="yes">
+<attribute name="VALUE" x="-78.74" y="-22.86" size="1.27" layer="96"/>
+<attribute name="NAME" x="-78.74" y="-25.4" size="1.27" layer="95"/>
+</instance>
+<instance part="SUPPLY1" gate="GND" x="-76.2" y="-48.26" smashed="yes">
+<attribute name="VALUE" x="-78.105" y="-51.435" size="1.778" layer="96"/>
+</instance>
+<instance part="FRAME3" gate="G$1" x="-129.54" y="-68.58" smashed="yes">
+<attribute name="DRAWING_NAME" x="87.63" y="-53.34" size="2.54" layer="94"/>
+<attribute name="LAST_DATE_TIME" x="87.63" y="-58.42" size="2.286" layer="94"/>
+<attribute name="SHEET" x="100.965" y="-63.5" size="2.54" layer="94"/>
+</instance>
 </instances>
 <busses>
